File: gpioexpander/gpioexpander.kicad_pcb (KiCad board)
At the start: 2 copper layers, 35.8 x 38.4 mm, 20 parts, among them J1 PWR/GND, J2 I2C, J3 Port 1, J4 Port 2, J5 Port 3, J6 Port 4, J7 Port 5, J8 ~INT, SW1 Action, U1 PCA9555PW,118

Commit message: Production run 1
Parts:
- H1, H2: footprint MountingHole:MountingHole_4.3mm_M4_Pad_Via -> MountingHole:MountingHole_3.2mm_M3_Pad
- U1: value PCA9555PW,118 -> PCA9555PW
- moved SW1 22.9 mm to (135.0, 72.5), turned to 180 degrees
- moved R1 20.2 mm to (134.5, 77.2), turned to 180 degrees
- moved J1 18.2 mm to (114.0, 61.1), turned to 0 degrees
- moved R3 16.3 mm to (122.8, 65.3), turned to 270 degrees
- moved J8 14.2 mm to (108.7, 72.0)
- moved R4 13.9 mm to (120.0, 65.3), turned to 270 degrees
- moved R7 11.0 mm to (120.0, 61.5)
- moved R5 10.9 mm to (117.3, 65.3), turned to 270 degrees
- moved H2 10.2 mm to (107.3, 62.2)
- moved H1 10.2 mm to (133.2, 62.2)
- moved R6 9.32 mm to (122.8, 61.5)
- moved J2 9.25 mm to (125.7, 61.6), turned to 0 degrees
- moved R2 8.79 mm to (109.6, 68.6)
- moved R8 6.42 mm to (117.3, 61.5)
Connections:
- net Net-(J2-Pad1) renamed /SCL
- net Net-(J2-Pad2) renamed /SDA
- net Net-(J3-Pad1) renamed /P1_1
- net Net-(J3-Pad2) renamed /P1_2
- net Net-(J3-Pad3) renamed /P1_3
- net Net-(J4-Pad1) renamed /P2_1
- net Net-(J4-Pad2) renamed /P2_2
- net Net-(J4-Pad3) renamed /P2_3
- net Net-(J5-Pad1) renamed /P3_1
- net Net-(J5-Pad2) renamed /P3_2
- net Net-(J5-Pad3) renamed /P3_3
- net Net-(J6-Pad1) renamed /P4_1
- net Net-(J6-Pad2) renamed /P4_2
- net Net-(J6-Pad3) renamed /P4_3
- net Net-(J7-Pad1) renamed /P5_1
- net Net-(J7-Pad2) renamed /P5_2
- net Net-(J7-Pad3) renamed /P5_3
- net Net-(J8-Pad1) renamed /~INT
- net Net-(R1-Pad1) renamed /SW1
Routing:
- net +3V3: track 40.0 -> 54.1 mm
- net /A0: track 25.3 -> 12.1 mm
- net GND: track 26.4 -> 15.0 mm
- net /SW1: track 28.2 -> 17.3 mm
- net /~INT: track 22.2 -> 13.8 mm
- net /A1: track 18.6 -> 13.9 mm
- net /SDA: track 11.6 -> 8.87 mm
- net /SCL: track 14.4 -> 12.4 mm
- net /A2: track 19.1 -> 19.9 mm
- net /P1_2: track 18.7 -> 18.0 mm
- net /P1_1: track 16.4 -> 17.0 mm
Other:
- board size 35.8 x 38.4 mm -> 35.8 x 37.3 mm
- board text added: "JNI2020 Expander board v1.2"
- board text removed: "JNI2020 Expander board v1"
