File: gpioexpander/gpioexpander.sch (KiCad schematic (older format))
At the start: 20 parts, among them J1 PWR/GND, J2 I2C, J3 Port 1, J4 Port 2, J5 Port 3, J6 Port 4, J7 Port 5, J8 ~INT, SW1 Action, U1 PCA9555PW

Commit message: Production run 1
Parts:
- H1, H2: footprint MountingHole:MountingHole_4.3mm_M4_Pad_Via -> MountingHole:MountingHole_3.2mm_M3_Pad
Connections:
- net ~INT: now reaches J8.1 (Pin_1), R2.1, U1.1 (~INT)
- net P3_1: now reaches J5.1 (Pin_1), U1.10 (IO0_6)
- net P3_2: now reaches J5.2 (Pin_2), U1.11 (IO0_7)
- net P3_3: now reaches J5.3 (Pin_3), U1.13 (IO1_0)
- net P4_1: now reaches J6.1 (Pin_1), U1.14 (IO1_1)
- net P4_2: now reaches J6.2 (Pin_2), U1.15 (IO1_2)
- net P4_3: now reaches J6.3 (Pin_3), U1.16 (IO1_3)
- net P5_1: now reaches J7.1 (Pin_1), U1.17 (IO1_4)
- net P5_2: now reaches J7.2 (Pin_2), U1.18 (IO1_5)
- net P5_3: now reaches J7.3 (Pin_3), U1.19 (IO1_6)
- net SW1: now reaches R1.1, SW1.1, U1.20 (IO1_7)
- net SCL: now reaches J2.1 (Pin_1), U1.22 (SCL)
- net SDA: now reaches J2.2 (Pin_2), U1.23 (SDA)
- net P1_1: now reaches J3.1 (Pin_1), U1.4 (IO0_0)
- net P1_2: now reaches J3.2 (Pin_2), U1.5 (IO0_1)
- net P1_3: now reaches J3.3 (Pin_3), U1.6 (IO0_2)
- net P2_1: now reaches J4.1 (Pin_1), U1.7 (IO0_3)
- net P2_2: now reaches J4.2 (Pin_2), U1.8 (IO0_4)
- net P2_3: now reaches J4.3 (Pin_3), U1.9 (IO0_5)
Other:
- moved on the sheet: R1
Changed lines of the file:
@@
 	4900 3100 7500 3100
 Wire Wire Line
-	4900 3300 7500 3200
+	4900 3300 5300 3300
 $Comp
 L power:GND #PWR0101
@@
 L power:GND #PWR0112
 U 1 1 5F54F050
-P 5050 4700
-F 0 "#PWR0112" H 5050 4450 50  0001 C CNN
-F 1 "GND" H 5055 4527 50  0000 C CNN
-F 2 "" H 5050 4700 50  0001 C CNN
-F 3 "" H 5050 4700 50  0001 C CNN
-	1    5050 4700
+P 5050 4750
+F 0 "#PWR0112" H 5050 4500 50  0001 C CNN
+F 1 "GND" H 5055 4577 50  0000 C CNN
+F 2 "" H 5050 4750 50  0001 C CNN
+F 3 "" H 5050 4750 50  0001 C CNN
+	1    5050 4750
 	1    0    0    -1
 $EndComp
@@
 L Device:R R1
 U 1 1 5F54E8D7
-P 5050 4550
-F 0 "R1" H 5120 4596 50  0000 L CNN
-F 1 "1K" H 5120 4505 50  0000 L CNN
-F 2 "Resistor_SMD:R_0603_1608Metric_Pad1.05x0.95mm_HandSolder" V 4980 4550 50  0001 C CNN
-F 3 "~" H 5050 4550 50  0001 C CNN
-F 4 "C21190" H 5050 4550 50  0001 C CNN "LCSC"
-	1    5050 4550
-	1    0    0    -1
-$EndComp
-Wire Wire Line
-	5050 4350 5050 4400
+P 5050 4600
+F 0 "R1" H 5120 4646 50  0000 L CNN
+F 1 "1K" H 5120 4555 50  0000 L CNN
+F 2 "Resistor_SMD:R_0603_1608Metric_Pad1.05x0.95mm_HandSolder" V 4980 4600 50  0001 C CNN
+F 3 "~" H 5050 4600 50  0001 C CNN
+F 4 "C21190" H 5050 4600 50  0001 C CNN "LCSC"
+	1    5050 4600
+	1    0    0    -1
+$EndComp
+Wire Wire Line
+	5050 4350 5050 4450
 Wire Wire Line
 	5050 4000 5050 4350
@@
 P 3050 2900
 F 0 "J8" H 2968 2663 50  0000 C CNN
-F 1 "~INT" H 2968 2761 50  0000 C CNN
+F 1 "~INT" H 3200 2900 50  0000 C CNN
 F 2 "Connector_PinHeader_2.54mm:PinHeader_1x01_P2.54mm_Vertical" H 3050 2900 50  0001 C CNN
 F 3 "~" H 3050 2900 50  0001 C CNN
@@
 F 0 "H1" V 3754 6300 50  0000 L CNN
 F 1 "MountingHole_Pad" V 3845 6300 50  0000 L CNN
-F 2 "MountingHole:MountingHole_4.3mm_M4_Pad_Via" H 3800 6150 50  0001 C CNN
+F 2 "MountingHole:MountingHole_3.2mm_M3_Pad" H 3800 6150 50  0001 C CNN
 F 3 "~" H 3800 6150 50  0001 C CNN
 	1    3800 6150
@@
 F 0 "H2" V 3754 6600 50  0000 L CNN
 F 1 "MountingHole_Pad" V 3845 6600 50  0000 L CNN
-F 2 "MountingHole:MountingHole_4.3mm_M4_Pad_Via" H 3800 6450 50  0001 C CNN
+F 2 "MountingHole:MountingHole_3.2mm_M3_Pad" H 3800 6450 50  0001 C CNN
 F 3 "~" H 3800 6450 50  0001 C CNN
 	1    3800 6450
@@
 Text Label 3800 4000 0    50   ~ 0
 A2
+Text Label 5000 4000 0    50   ~ 0
+SW1
+Text Label 3450 2900 0    50   ~ 0
+~INT
+Text Label 3400 2400 0    50   ~ 0
+SCL
+Text Label 3400 2500 0    50   ~ 0
+SDA
+Text Label 8150 2400 0    50   ~ 0
+P1_1
+Text Label 8150 2500 0    50   ~ 0
+P1_2
+Text Label 8150 2600 0    50   ~ 0
+P1_3
+Text Label 7500 2700 0    50   ~ 0
+P2_1
+Text Label 7500 2800 0    50   ~ 0
+P2_2
+Text Label 7500 2900 0    50   ~ 0
+P2_3
+Text Label 6650 3000 0    50   ~ 0
+P3_1
+Text Label 6650 3100 0    50   ~ 0
+P3_2
+Text Label 6650 3200 0    50   ~ 0
+P3_3
+Wire Wire Line
+	5300 3300 5300 3200
+Wire Wire Line
+	5300 3200 7500 3200
+Text Label 6150 3400 0    50   ~ 0
+P4_1
+Text Label 6150 3500 0    50   ~ 0
+P4_2
+Text Label 6150 3600 0    50   ~ 0
+P4_3
+Text Label 5500 3700 0    50   ~ 0
+P5_1
+Text Label 5500 3800 0    50   ~ 0
+P5_2
+Text Label 5500 3900 0    50   ~ 0
+P5_3
 $EndSCHEMATC
