File: gpioexpander4/gpioexpander4.kicad_pcb (KiCad board)
At the start: 2 copper layers, 39.6 x 40.6 mm, 21 parts, among them J1 PWR, J2 I2C, J3 Port 1, J4 Port 2, J5 Port 3, J6 Port 4, J7 Port 5, J8 ~INT, SW1 Action, U1 MCP23017-E/SP

Commit message: Production run 1
Parts:
- added G***: LOGO, bre:brain, F.Cu at (136.7, 77.3)
- added J9: Reset, Connector_PinHeader_2.54mm:PinHeader_1x02_P2.54mm_Vertical, F.Cu at (112.3, 76.3)
- added R10: 1K, Resistor_SMD:R_0805_2012Metric_Pad1.15x1.40mm_HandSolder, F.Cu at (118.0, 76.5)
- H1, H2: footprint MountingHole:MountingHole_4.3mm_M4_Pad -> MountingHole:MountingHole_3.2mm_M3_Pad
- moved H1 0.81 mm to (139.7, 53.2)
- moved H2 0.46 mm to (111.4, 82.8)
Connections:
- U1 pad 18: +3V3 -> /~RESET
Routing:
- net /~RESET: track 0.00 -> 20.3 mm
- net +3V3: track 39.5 -> 38.0 mm
Other:
- board text added: "GPIO Expander v4.1 JN2020"
- board text removed: "GPIO Expander v4 JN2020"
