File: gpioexpander5/gpioexpander5.kicad_pcb (KiCad board)
At the start: 2 copper layers, 39.6 x 40.6 mm, 24 parts, among them J1 PWR, J2 I2C, J3 Port 1, J4 Port 2, J5 Port 3, J6 Port 4, J7 Port 5, J8 ~INT, J9 RESET, SW1 Action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

Commit message: Add hi/lo ot addr
Other:
- board text added: "Hi"
- board text added: "Lo"

Commit message: gpioexpander v5.1
4 pin headers document hi/lo side
Parts:
- removed G***: LOGO, br:brain
- removed J8: ~INT, Connector_PinHeader_2.54mm:PinHeader_1x02_P2.54mm_Vertical
- removed J9: RESET, Connector_PinHeader_2.54mm:PinHeader_1x02_P2.54mm_Vertical
- J1: value PWR -> RST+INT; footprint Connector_PinHeader_2.54mm:PinHeader_1x02_P2.54mm_Vertical -> Connector_PinHeader_2.54mm:PinHeader_1x04_P2.54mm_Vertical
- J2: footprint Connector_PinHeader_2.54mm:PinHeader_1x02_P2.54mm_Vertical -> Connector_PinHeader_2.54mm:PinHeader_1x04_P2.54mm_Vertical
- moved J1 22.8 mm to (142.1, 67.9), turned to 0 degrees
- moved J2 3.42 mm to (120.4, 84.7), turned to 90 degrees
Connections:
- J1 pad 1: +3V3 -> /INTA
- J1 pad 2: GND -> /INTB
Routing:
- net /~RESET: track 21.6 -> 25.5 mm
- net /SDA: track 18.4 -> 20.6 mm
- net /A1: track 22.4 -> 20.8 mm
- net /SCK: track 22.6 -> 21.2 mm
- net /INTB: track 19.9 -> 18.9 mm
- net /A0: track 23.6 -> 24.5 mm
- net /INTA: track 19.1 -> 18.4 mm
Other:
- board text added: "GPIO Expander V5.1 JN 2020"
- board text added: "PWR"
- board text added: "RST"
- board text removed: "GPIO Expander V5 JN 2020"
- board text removed: "Power In"
- board text removed: "Reset"
