File: gpioexpander5/gpioexpander5.sch (KiCad schematic (older format))
At the start: 23 parts, among them J1 PWR, J2 I2C, J3 Port 1, J4 Port 2, J5 Port 3, J6 Port 4, J7 Port 5, J8 ~INT, J9 RESET, SW1 Action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

Commit message: gpioexpander v5.1
4 pin headers document hi/lo side
Parts:
- removed J1: PWR, Connector_PinHeader_2.54mm:PinHeader_1x02_P2.54mm_Vertical, symbol Connector_Generic:Conn_01x02
- removed J8: ~INT, Connector_PinHeader_2.54mm:PinHeader_1x02_P2.54mm_Vertical, symbol Connector_Generic:Conn_01x02
- removed J9: RESET, Connector_PinHeader_2.54mm:PinHeader_1x02_P2.54mm_Vertical, symbol Connector:Conn_01x02_Male
- added J1: RST+INT, Connector_PinHeader_2.54mm:PinHeader_1x04_P2.54mm_Vertical, symbol Connector_Generic:Conn_01x04
- J2: footprint Connector_PinHeader_2.54mm:PinHeader_1x02_P2.54mm_Vertical -> Connector_PinHeader_2.54mm:PinHeader_1x04_P2.54mm_Vertical; symbol Connector_Generic:Conn_01x02 -> Connector_Generic:Conn_01x04
Connections:
- net +3V3: now also J2.4 (Pin_4)
- net GND: now also J2.3 (Pin_3), J1.4 (Pin_4)
- net INTA: now also J1.1 (Pin_1)
- net INTB: now also J1.2 (Pin_2)
- net ~RESET: now also J1.3 (Pin_3)
Other:
- moved on the sheet: R10, R2, R3
